File: DI-Lambda-UNO/DI-Lambda-UNO-bottom/DI-Lambda-UNO-bottom.kicad_pcb (KiCad board)
At the start: 2 copper layers, 118.4 x 128.1 mm, 53 parts, among them J1 Conn_02x04_Odd_Even, J15 CONN_01X06, J16 CONN_01X06, J17 CONN_02X03, J18 USB_OTG, J2 Conn_01X01, J3 Conn_02x04_Odd_Even, J4 Conn_01X01, J5 Conn_01x01, J6 Conn_02x03_Odd_Even, J7 Conn_02x03_Odd_Even, J8 Conn_02x04_Odd_Even, J9 Conn_02x04_Odd_Even, Q1 Q_NMOS_GSD, SW1 RESET, U2 USBLC6-2SC6, U3 ATMEGA32U4-MU, U4 3.3v LDO, U5 AP3032, Y1 8Mhz

Commit message: Version 1.5
Parts:
- removed C1: 0.1uF, Capacitor_SMD:C_0603_1608Metric
- removed C10, C11, C8, C9: 0.1uF 25v, Capacitor_SMD:C_0603_1608Metric
- removed C2, C3: 22pF 25V, Capacitor_SMD:C_0603_1608Metric
- removed C4: 4.7uF 25V, Capacitor_SMD:C_0603_1608Metric
- removed C5: 1uF 25V, Capacitor_SMD:C_0603_1608Metric
- removed J17: CONN_02X03, Female_socket_pitch254_smt_through-board:Pin_Header_Straight_2x03_Pitch2.54mm_SMD_wide
- removed R1, R5, R9: 4.7k, Resistor_SMD:R_0603_1608Metric
- removed R2: 330R, Resistor_SMD:R_0603_1608Metric
- removed SW1: RESET, Buttons_Switches_SMD:SW_SPST_TL3342
- removed U3: ATMEGA32U4-MU, Housings_QFP:TQFP-44_10x10mm_Pitch0.8mm
- removed U5: AP3032, TO_SOT_Packages_SMD:SOT-23-6
- removed Y1: 8Mhz, Crystals:Crystal_SMD_HC49-SD
- added U1: AP3015, Package_TO_SOT_SMD:SOT-23-5, F.Cu at (154.6, 69.4)
- J2, J4: value Conn_01X01 -> Conn_02x02_Odd_Even; footprint Measurement_Points:Measurement_Point_Round-SMD-Pad_Small -> Connector_PinSocket_2.54mm:PinSocket_2x02_P2.54mm_Vertical_SMD
- U4: footprint TO_SOT_Packages_SMD:SOT-23 -> Package_TO_SOT_SMD:SOT-89-3
- moved J18 129.8 mm to (146.0, 167.4), turned to 0 degrees
- moved L1 96.8 mm to (141.0, 145.6), turned to 270 degrees
- moved L2 92.3 mm to (161.4, 147.9), turned to 90 degrees
- moved L3 91.5 mm to (159.7, 147.9), turned to 90 degrees
- moved R10 87.8 mm to (145.0, 145.6), turned to 270 degrees
- moved R11 87.7 mm to (146.9, 145.6), turned to 270 degrees
- moved F1 85.2 mm to (141.0, 141.3), turned to 270 degrees
- moved U2 79.7 mm to (145.9, 141.3), turned to 270 degrees
- moved C13 62.5 mm to (143.3, 140.4)
- moved J2 31.2 mm to (161.9, 76.2), turned to 90 degrees
- moved J4 25.6 mm to (138.9, 76.2), turned to 270 degrees
- moved C6 15.1 mm to (155.7, 76.2)
- moved C7 11.4 mm to (152.7, 79.6), turned to 180 degrees
- moved R14 10.3 mm to (151.7, 65.6), turned to 90 degrees
- moved L4 9.88 mm to (158.2, 69.4)
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Connections:
- net Net-(J18-Pad2) renamed /DI_N
- net Net-(J18-Pad3) renamed /DI_P
- J1 pad 1: Net-(J1-Pad1) -> GND
- J1 pad 2: Net-(J1-Pad2) -> GND
- J1 pad 3: Net-(J1-Pad3) -> GND
- J1 pad 4: Net-(J1-Pad4) -> GND
- J1 pad 5: Net-(J1-Pad5) -> GND
- J1 pad 6: Net-(J1-Pad6) -> GND
- J1 pad 7: Net-(J1-Pad7) -> GND
- J1 pad 8: Net-(J1-Pad8) -> GND
- J2 pad 1: /RX -> /SCL
- J3 pad 1: Net-(J3-Pad1) -> GND
- J3 pad 2: Net-(J3-Pad2) -> GND
- J3 pad 3: Net-(J3-Pad3) -> GND
- J3 pad 4: Net-(J3-Pad4) -> GND
- J3 pad 5: Net-(J3-Pad5) -> GND
- J3 pad 6: Net-(J3-Pad6) -> GND
- J3 pad 7: Net-(J3-Pad7) -> GND
- J3 pad 8: Net-(J3-Pad8) -> GND
- J4 pad 1: /TX -> /D_N
- J6 pad 1: Net-(J6-Pad1) -> GND
- J6 pad 2: Net-(J6-Pad2) -> GND
- J6 pad 3: Net-(J6-Pad3) -> GND
- J6 pad 4: Net-(J6-Pad4) -> GND
- J6 pad 5: Net-(J6-Pad5) -> GND
- J6 pad 6: Net-(J6-Pad6) -> GND
- J7 pad 1: Net-(J7-Pad1) -> GND
- J7 pad 2: Net-(J7-Pad2) -> GND
- J7 pad 3: Net-(J7-Pad3) -> GND
- J7 pad 4: Net-(J7-Pad4) -> GND
- J7 pad 5: Net-(J7-Pad5) -> GND
- J7 pad 6: Net-(J7-Pad6) -> GND
- J8 pad 1: Net-(J8-Pad1) -> GND
- J8 pad 2: Net-(J8-Pad2) -> GND
- J8 pad 3: Net-(J8-Pad3) -> GND
- J8 pad 4: Net-(J8-Pad4) -> GND
- J8 pad 5: Net-(J8-Pad5) -> GND
- J8 pad 6: Net-(J8-Pad6) -> GND
- J8 pad 7: Net-(J8-Pad7) -> GND
- J8 pad 8: Net-(J8-Pad8) -> GND
- J9 pad 1: Net-(J9-Pad1) -> GND
- J9 pad 2: Net-(J9-Pad2) -> GND
- J9 pad 3: Net-(J9-Pad3) -> GND
- J9 pad 4: Net-(J9-Pad4) -> GND
- J9 pad 5: Net-(J9-Pad5) -> GND
- J9 pad 6: Net-(J9-Pad6) -> GND
- J9 pad 7: Net-(J9-Pad7) -> GND
- J9 pad 8: Net-(J9-Pad8) -> GND
- R10 pad 1: Net-(R10-Pad1) -> /D_N
- R11 pad 1: Net-(R11-Pad1) -> /D_P
- U2 pad 1: Net-(R11-Pad1) -> /D_P
- U2 pad 3: Net-(R10-Pad1) -> /D_N
- U2 pad 4: Net-(R10-Pad1) -> /D_N
- U2 pad 6: Net-(R11-Pad1) -> /D_P
Routing:
- net GND: track 121.9 -> 26.1 mm, vias 22 -> 10
- net /D_P: track 0.00 -> 73.2 mm
- net /D_N: track 0.00 -> 68.0 mm
- net /VCC: track 195.6 -> 148.7 mm, vias 7 -> 0
- net /VBUS: track 64.2 -> 106.6 mm, vias 7 -> 0
- net /RST: track 35.0 -> 0.00 mm, vias 2 -> 0
- net Net-(R11-Pad1): track 28.6 -> 0.00 mm, vias 2 -> 0
- net Net-(R10-Pad1): track 28.6 -> 0.00 mm, vias 2 -> 0
- net /MOSI: track 26.6 -> 0.00 mm, vias 1 -> 0
- net /TX: track 18.7 -> 0.00 mm, vias 2 -> 0
- net /LED_PWM: track 44.4 -> 26.5 mm, vias 2 -> 0
- net /RX: track 17.8 -> 0.00 mm, vias 2 -> 0
- net /VLED: track 31.4 -> 14.7 mm, vias 2 -> 0
- net /MISO: track 14.8 -> 0.00 mm, vias 1 -> 0
- net /SCK: track 14.7 -> 0.00 mm, vias 1 -> 0
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Other:
- board size 118.4 x 128.1 mm -> 38.2 x 128 mm
- board text removed: "RESET"
- board text removed: "RX"
- board text removed: "TX"

Commit message: Version 1.6
Parts:
- added C1: 1uF 16v, Capacitor_SMD:C_0603_1608Metric, F.Cu at (155.5, 65.2)
- added Q2: AO3401, Package_TO_SOT_SMD:SOT-23, F.Cu at (152.8, 58.0)
- added R1: 4.7k, Resistor_SMD:R_0603_1608Metric, F.Cu at (155.5, 57.5)
- C12, C13, C6, C7: value 4.7uF 25v -> 4.7uF 6.3v
- C14: value 4.7uF 25v -> 1uF 16v
- D3: footprint Diodes_SMD:D_SMA_Standard -> Diode_SMD:D_SMA
- F1: footprint Fuse_Holders_and_Fuses:Fuse_SMD1206_Reflow -> Fuse:Fuse_1206_3216Metric
- J18: footprint Connectors_USB:USB_Micro-B_Molex-105017-0001 -> Connector_USB:USB_Micro-B_Molex-105017-0001
- L4: footprint Inductors:Inductor_Taiyo-Yuden_NR-30xx -> Inductor_SMD:L_Taiyo-Yuden_NR-40xx
- Q1: value Q_NMOS_GSD -> AO3400
- U2: footprint TO_SOT_Packages_SMD:SOT-23-6 -> Package_TO_SOT_SMD:SOT-23-6
- U4: footprint Package_TO_SOT_SMD:SOT-89-3 -> Package_TO_SOT_SMD:SOT-223-3_TabPin2
- moved R3 4.38 mm to (150.2, 58.5), turned to 90 degrees
- moved Q1 3.90 mm to (158.0, 57.7)
- moved U4 1.75 mm to (150.4, 76.2)
- moved C7 1.19 mm to (152.3, 80.7)
- moved C14 1.08 mm to (153.9, 65.2)
- moved R13 1.08 mm to (152.3, 65.2)
- moved R14 1.08 mm to (150.7, 65.2)
- moved D3 1.00 mm to (158.2, 63.1)
- moved J18 0.90 mm to (145.9, 166.5)
- moved U2 0.90 mm to (145.9, 142.2)
- moved C13 0.83 mm to (143.3, 141.3), turned to 90 degrees
- moved C12 0.75 mm to (151.9, 68.7)
- moved U1 0.75 mm to (154.5, 68.7)
- moved L4 0.67 mm to (158.7, 68.9)
- moved J15 0.10 mm to (150.4, 153.6)
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Connections:
- C13 pad 1: GND -> /VBUS
- C13 pad 2: /VBUS -> GND
- C14 pad 1: /VLED -> /12v
- D3 pad 1: /VLED -> /12v
- J16 pad 5: /GLED -> GND
- Q1 pad 3: /GLED -> Net-(Q1-Pad3)
- R13 pad 1: /VLED -> /12v
Routing:
- net /12v: track 0.00 -> 17.1 mm
- net /VLED: track 14.7 -> 5.93 mm
- net GND: track 26.1 -> 34.2 mm, vias 10 -> 15
- net /VBUS: track 106.6 -> 113.7 mm
- net Net-(J18-Pad5): track 23.8 -> 30.5 mm
- net /LED_PWM: track 26.5 -> 31.0 mm
- net Net-(Q1-Pad3): track 0.00 -> 4.48 mm
- net /D_P: track 73.2 -> 77.2 mm
- net /D_N: track 68.0 -> 71.8 mm
- net /GLED: track 2.40 -> 0.00 mm
- net Net-(J18-Pad6): track 39.6 -> 41.7 mm
- net /VCC: track 148.7 -> 149.9 mm
- net /SW: track 4.96 -> 5.88 mm
Other:
- board text added: "DI-Lambda UNO v1.6"
- board text removed: "DI-Lambda UNO v1.5"

Commit message: More missing fotprints
Parts:
- R103: renamed from R1; value 4.7k -> 4.75k
- R104: renamed from R3; value 4.7k -> 4.75k
- R105: renamed from R13; value 59K -> 42.2k
- R106: renamed from R14; value 1K -> 4.75k
- moved Q102 143.6 mm to (19.9, 18.4)
- moved R103 137.6 mm to (23.4, 18.8), turned to 180 degrees
- moved C102 137.6 mm to (24.4, 35.0)
- moved L103 137.6 mm to (28.4, 106.8)
- moved R102 137.6 mm to (13.7, 104.5)
- moved R106 137.6 mm to (19.4, 24.1)
- moved C103 137.6 mm to (21.0, 39.5)
- moved C104 137.6 mm to (24.2, 24.1)
- moved C105 137.6 mm to (20.6, 27.5)
- moved C106 137.6 mm to (22.6, 24.1)
- moved D101 137.6 mm to (26.9, 21.9)
- moved F101 137.6 mm to (9.75, 100.1)
- moved J101 137.6 mm to (14.7, 125.3)
- moved J102 137.6 mm to (19.1, 112.4)
- moved J103 137.6 mm to (3.30, 15.0)
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- renumbered C13 to C101, C6 to C102, C7 to C103, C1 to C104, C12 to C105, C14 to C106, D3 to D101, F1 to F101, J18 to J101, J15 to J102, J1 to J103, J3 to J104, J4 to J105, J2 to J106, J5 to J107, J6 to J108, J7 to J109, J8 to J110, J9 to J111, J16 to J112, L1 to L101, L2 to L102, L3 to L103, L4 to L104, MK2 to MK101, MK1 to MK102, MK3 to MK103, MK4 to MK104, Q2 to Q101, Q1 to Q102, R11 to R101, R10 to R102, U2 to U101, U4 to U102, U1 to U103
Connections:
- J103 pad 1: GND -> Net-(J103-Pad1)
- J103 pad 2: GND -> Net-(J103-Pad2)
- J103 pad 3: GND -> Net-(J103-Pad3)
- J103 pad 4: GND -> Net-(J103-Pad4)
- J103 pad 5: GND -> Net-(J103-Pad5)
- J103 pad 6: GND -> Net-(J103-Pad6)
- J103 pad 7: GND -> Net-(J103-Pad7)
- J103 pad 8: GND -> Net-(J103-Pad8)
- J104 pad 1: GND -> Net-(J104-Pad1)
- J104 pad 2: GND -> Net-(J104-Pad2)
- J104 pad 3: GND -> Net-(J104-Pad3)
- J104 pad 4: GND -> Net-(J104-Pad4)
- J104 pad 5: GND -> Net-(J104-Pad5)
- J104 pad 6: GND -> Net-(J104-Pad6)
- J104 pad 7: GND -> Net-(J104-Pad7)
- J104 pad 8: GND -> Net-(J104-Pad8)
- J108 pad 1: GND -> Net-(J108-Pad1)
- J108 pad 2: GND -> Net-(J108-Pad2)
- J108 pad 3: GND -> Net-(J108-Pad3)
- J108 pad 4: GND -> Net-(J108-Pad4)
- J108 pad 5: GND -> Net-(J108-Pad5)
- J108 pad 6: GND -> Net-(J108-Pad6)
- J109 pad 1: GND -> Net-(J109-Pad1)
- J109 pad 2: GND -> Net-(J109-Pad2)
- J109 pad 3: GND -> Net-(J109-Pad3)
- J109 pad 4: GND -> Net-(J109-Pad4)
- J109 pad 5: GND -> Net-(J109-Pad5)
- J109 pad 6: GND -> Net-(J109-Pad6)
- J110 pad 1: GND -> Net-(J110-Pad1)
- J110 pad 2: GND -> Net-(J110-Pad2)
- J110 pad 3: GND -> Net-(J110-Pad3)
- J110 pad 4: GND -> Net-(J110-Pad4)
- J110 pad 5: GND -> Net-(J110-Pad5)
- J110 pad 6: GND -> Net-(J110-Pad6)
- J110 pad 7: GND -> Net-(J110-Pad7)
- J110 pad 8: GND -> Net-(J110-Pad8)
- J111 pad 1: GND -> Net-(J111-Pad1)
- J111 pad 2: GND -> Net-(J111-Pad2)
- J111 pad 3: GND -> Net-(J111-Pad3)
- J111 pad 4: GND -> Net-(J111-Pad4)
- J111 pad 5: GND -> Net-(J111-Pad5)
- J111 pad 6: GND -> Net-(J111-Pad6)
- J111 pad 7: GND -> Net-(J111-Pad7)
- J111 pad 8: GND -> Net-(J111-Pad8)
- Q101 pad 2: /VLED -> /12v
- Q101 pad 3: /12v -> /VLED
- R101 pad 1: /D_P -> /_D_P
- R102 pad 1: /D_N -> /_D_N
- U101 pad 4: /D_N -> /_D_N
- U101 pad 6: /D_P -> /_D_P
Routing:
- net GND: track 34.2 -> 109.0 mm, vias 15 -> 10
- net /LED_PWM: track 31.0 -> 22.8 mm
- net /D_P: track 77.2 -> 71.8 mm
- net /D_N: track 71.8 -> 66.7 mm
- net /SCL: track 123.3 -> 127.2 mm
- net /VCC: track 149.9 -> 153.7 mm
- net /VBUS: track 113.7 -> 110.6 mm
- net Net-(J101-Pad6): track 41.7 -> 44.4 mm
- net /VLED: track 5.93 -> 3.32 mm
- net /12v: track 17.1 -> 14.8 mm
- net /SDA: track 126.5 -> 128.1 mm
- net /_D_P: track 0.00 -> 1.42 mm
- net /_D_N: track 0.00 -> 1.42 mm
- net /DI_N: track 20.8 -> 20.2 mm
Other:
- rule pad_to_mask_clearance: 0.2 -> 0.07
- board text added: "DI-Lambda UNO v1.7"
- board text removed: "DI-Lambda UNO v1.6"
