File: DI-Lambda-UNO/DI-Lambda-UNO-top/DI-Lambda-UNO-top.kicad_pcb (KiCad board)
At the start: 2 copper layers, 38.2 x 128 mm, 37 parts, among them J1 Conn_02x04_Odd_Even, J10 Conn_02x02_Odd_Even, J11 Conn_02x02_Odd_Even, J12 Conn_01x05, J13 Conn_01x11, J17 CONN_02X03, J2 Conn_01X01, J3 Conn_02x04_Odd_Even, J4 Conn_01X01, J5 Conn_01x11, J6 Conn_02x03_Odd_Even, J7 Conn_02x03_Odd_Even, J8 Conn_02x04_Odd_Even, J9 Conn_02x04_Odd_Even, SW2 SW_BLANK, SW3 SW_SAMPLE, SW4 SW_MODE, U1 LCD_1.44_ST7735, U3 ATMEGA32U4-MU, Y1 8Mhz

Commit message: Version 1.6
Parts:
- removed J12: Conn_01x05, Connector_PinHeader_2.54mm:PinHeader_1x05_P2.54mm_Vertical
- removed J13, J5: Conn_01x11, Connector_PinHeader_2.54mm:PinHeader_1x11_P2.54mm_Vertical
- removed J17: CONN_02X03, Connector_PinSocket_2.54mm:PinSocket_2x03_P2.54mm_Vertical_SMD
- removed R1: 4.7k, Resistor_SMD:R_0603_1608Metric
- removed U3: ATMEGA32U4-MU, Housings_QFP:TQFP-44_10x10mm_Pitch0.8mm
- added C12: 4.7uF 25V, Capacitor_SMD:C_0603_1608Metric, F.Cu at (147.4, 74.1)
- added C13: 0.1uF 25v, Capacitor_SMD:C_0603_1608Metric, F.Cu at (152.4, 87.7)
- added C6: 4.7uF 25V, Capacitor_SMD:C_0603_1608Metric, F.Cu at (152.4, 89.2)
- added C7: 4.7uF 25V, Capacitor_SMD:C_0603_1608Metric, F.Cu at (139.0, 71.7)
- added J14: Conn_01x05, test_points:Testpoint_1x05_P2.54mm_mixed, F.Cu at (153.3, 166.8)
- added MK2: Mounting_Hole, Mounting-holes:Mounting-Hole-SMT-nut-M3-4.3mm, B.Cu at (161.8, 96.1)
- added MK3: Mounting_Hole, Mounting-holes:Mounting-Hole-SMT-nut-M3-4.3mm, B.Cu at (139.0, 96.1)
- added MK4: Mounting_Hole, Mounting-holes:Mounting-Hole-SMT-nut-M3-4.3mm, B.Cu at (134.6, 44.5)
- added MK5: Mounting_Hole, Mounting-holes:Mounting-Hole-SMT-nut-M3-4.3mm, B.Cu at (166.2, 44.5)
- added MK6: Mounting_Hole, DI-Lambda-module-tabs:Button_mounts_x3, F.Cu at (150.4, 44.5)
- added R2: 390R, Resistor_SMD:R_0603_1608Metric, F.Cu at (141.2, 88.9)
- added R8: 1.5K, Resistor_SMD:R_0603_1608Metric, F.Cu at (157.5, 76.8)
- added U2: STM32F103C8Tx, Package_QFP:LQFP-48_7x7mm_P0.5mm, F.Cu at (149.9, 81.6)
- C2, C3: value 22pF 25V -> 20pF 25V
- C4: value 4.7uF 25V -> 0.1uF 25v
- C5: value 1uF 25V -> 4.7uF 25V
- J10, J11: footprint Connector_PinSocket_2.54mm:PinSocket_2x02_P2.54mm_Vertical_SMD -> Connector_PinHeader_2.54mm:PinHeader_2x02_P2.54mm_Vertical_SMD
- J2, J4: value Conn_01X01 -> Conn_02x02_Odd_Even; footprint Measurement_Points:Measurement_Point_Round-SMD-Pad_Small -> Connector_PinHeader_2.54mm:PinHeader_2x02_P2.54mm_Vertical_SMD
- MK1: footprint DI-Lambda-module-tabs:Cuvette-cutout-top -> Cuvette-holder:Cuvette-cutout-top
- SW2: value SW_BLANK -> SW_SAMPLE; footprint Button_Switch_SMD:SW_SPST_PTS645 -> Button_Switch_SMD:SW_SPST_B3SL-1002P
- SW3: value SW_SAMPLE -> SW_MODE; footprint Button_Switch_SMD:SW_SPST_PTS645 -> Button_Switch_SMD:SW_SPST_B3SL-1002P
- SW4: value SW_MODE -> SW_BLANK; footprint Button_Switch_SMD:SW_SPST_PTS645 -> Button_Switch_SMD:SW_SPST_B3SL-1002P
- Y1: footprint Crystals:Crystal_SMD_HC49-SD -> Crystal:Crystal_SMD_HC49-SD
- moved J2 43.3 mm to (161.9, 139.2), turned to 90 degrees
- moved J4 39.8 mm to (138.9, 139.2), turned to 90 degrees
- moved C9 21.6 mm to (147.4, 75.6), turned to 0 degrees
- moved C8 19.7 mm to (143.8, 83.1)
- moved C11 18.8 mm to (143.8, 78.0), turned to 90 degrees
- moved C2 17.9 mm to (136.9, 78.0)
- moved C5 14.4 mm to (150.6, 66.6), turned to 180 degrees
- moved C10 13.6 mm to (156.0, 79.1)
- moved R9 12.8 mm to (143.7, 62.0), turned to 0 degrees
- moved Y1 11.9 mm to (140.4, 81.4), turned to 270 degrees
- moved C1 11.7 mm to (150.4, 69.1), turned to 0 degrees
- moved C4 10.6 mm to (146.4, 89.8), turned to 0 degrees
- moved U1 10.5 mm to (150.4, 64.1)
- moved R5 10.3 mm to (143.7, 63.7), turned to 180 degrees
- moved C3 10.0 mm to (136.9, 84.7), turned to 90 degrees
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Connections:
- C1 pad 1: GND -> /VCC
- C1 pad 2: /RST -> GND
- C4 pad 1: /VBUS -> /nRST
- C5 pad 1: /VCC -> GND
- C5 pad 2: GND -> /VCC
- J10 pad 1: /DP -> /DN
- J10 pad 2: /DN -> /DP
- J10 pad 3: /LED_PWM -> /VBUS
- J10 pad 4: /VBUS -> /LED_PWM
- J11 pad 1: /VCC -> /SCL
- J11 pad 2: /SCL -> /VCC
- J11 pad 3: GND -> /SDA
- J11 pad 4: /SDA -> GND
- J2 pad 1: /RX -> Net-(J2-Pad1)
- J4 pad 1: /TX -> Net-(J4-Pad1)
- R4 pad 2: /BLANK -> /SAMPLE
- R6 pad 2: /SAMPLE -> /MODE
- R7 pad 2: /MODE -> /BLANK
Routing:
- net GND: track 41.3 -> 164.0 mm, vias 12 -> 13
- net /VCC: track 98.0 -> 205.4 mm, vias 4 -> 8
- net /SWDCLK: track 0.00 -> 96.6 mm, vias 0 -> 2
- net /nRST: track 0.00 -> 93.3 mm
- net /SWDIO: track 0.00 -> 93.1 mm, vias 0 -> 2
- net /MODE: track 63.8 -> 21.4 mm, vias 2 -> 0
- net /VBUS: track 23.4 -> 0.00 mm, vias 2 -> 0
- net /BLANK: track 52.0 -> 29.8 mm, vias 2 -> 0
- net /SAMPLE: track 45.2 -> 23.9 mm, vias 2 -> 0
- net /LCD_LED: track 32.2 -> 14.5 mm
- net /LED_PWM: track 42.1 -> 25.8 mm
- net /RST: track 14.9 -> 0.00 mm, vias 2 -> 0
- net /SCL: track 36.9 -> 24.3 mm
- net /SDA: track 43.1 -> 31.6 mm
- net /RX: track 11.4 -> 0.00 mm, vias 2 -> 0
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Other:
- outline, holes or cut-outs redrawn
- net class Default: clearance 0.2 -> 0.15; trace_width 0.25 -> 0.15; via_dia 0.8 -> 0.6; via_drill 0.4 -> 0.3
- net class POWER added: clearance 0.2, trace_width 0.3, via_dia 0.6, via_drill 0.3
- rule pad_to_mask_clearance: 0.2 -> 0.07
- rule trace_clearance: 0.2 -> 0.15
- rule trace_min: 0.2 -> 0.15
- board text added: "DI-Lambda UNO v1.6"
- board text removed: "DI-Lambda UNO v1.5"
- board text removed: "RX"
- board text removed: "TX"

Commit message: More missing fotprints
Parts:
- removed J10, J11, J2, J4: Conn_02x02_Odd_Even, Connector_PinHeader_2.54mm:PinHeader_2x02_P2.54mm_Vertical_SMD
- added J203: Conn_02x02_Odd_Even, Connector_PinHeader_2.54mm:PinHeader_2x02_P2.54mm_Vertical_SMD_vias, F.Cu at (7.60, 25.0)
- added J204: Conn_02x02_Odd_Even, Connector_PinHeader_2.54mm:PinHeader_2x02_P2.54mm_Vertical_SMD_vias, F.Cu at (30.6, 25.0)
- added J207: Conn_02x02_Odd_Even, Connector_PinHeader_2.54mm:PinHeader_2x02_P2.54mm_Vertical_SMD_vias, F.Cu at (30.6, 98.0)
- added J208: Conn_02x02_Odd_Even, Connector_PinHeader_2.54mm:PinHeader_2x02_P2.54mm_Vertical_SMD_vias, F.Cu at (7.60, 98.0)
- C201: renamed from C5; value 4.7uF 25V -> 4.7uF 6.3v
- C203: renamed from C2; value 20pF 25V -> 10pF 25V
- C204: renamed from C3; value 20pF 25V -> 10pF 25V
- C205: renamed from C6; value 4.7uF 25V -> 4.7uF 6.3v
- C206: renamed from C7; value 4.7uF 25V -> 4.7uF 6.3v
- C207: renamed from C12; value 4.7uF 25V -> 4.7uF 6.3v
- R203: renamed from R5; value 4.7k -> 4.75K
- R204: renamed from R9; value 4.7k -> 4.75K
- R206: renamed from R4; value 220R -> 1.5K
- R207: renamed from R6; value 220R -> 1.5K
- R208: renamed from R7; value 220R -> 1.5K
- moved MK201 137.8 mm to (19.1, 2.50)
- moved C202 137.6 mm to (15.2, 48.7)
- moved C204 137.6 mm to (5.67, 43.6)
- moved C206 137.6 mm to (7.70, 30.5)
- moved C212 137.6 mm to (24.7, 38.0)
- moved MK203 137.6 mm to (7.70, 54.9)
- moved R201 137.6 mm to (26.2, 34.0)
- moved R203 137.6 mm to (12.4, 22.5)
- moved R204 137.6 mm to (12.4, 20.8)
- moved R205 137.6 mm to (26.2, 35.6)
- moved C201 137.6 mm to (19.3, 25.4)
- moved C203 137.6 mm to (5.66, 36.8)
- moved C205 137.6 mm to (21.1, 48.0)
- moved C207 137.6 mm to (16.1, 32.9)
- moved C208 137.6 mm to (19.1, 27.9)
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- renumbered C4 to C202, C1 to C208, C13 to C209, C8 to C210, C9 to C211, C10 to C212, C11 to C213, J1 to J201, J3 to J202, J6 to J205, J7 to J206, J8 to J209, J9 to J210, J14 to J211, MK6 to MK201, MK2 to MK202, MK3 to MK203, MK4 to MK204, MK5 to MK205, MK1 to MK206, R3 to R201, R2 to R202, R8 to R205, SW2 to SW201, SW3 to SW202, SW4 to SW203, U1 to U201, U2 to U202, Y1 to Y201
Connections:
- U202 pad 27: Net-(U2-Pad27) -> /LED_PWM
- U202 pad 28: Net-(U2-Pad28) -> /MODE
- U202 pad 29: Net-(U2-Pad29) -> /SAMPLE
- U202 pad 38: /LED_PWM -> Net-(U202-Pad38)
- U202 pad 39: /MODE -> Net-(U202-Pad39)
- U202 pad 40: /SAMPLE -> Net-(U202-Pad40)
Routing:
- net /LED_PWM: track 25.8 -> 37.1 mm, vias 0 -> 2
- net /SAMPLE: track 23.9 -> 34.4 mm, vias 0 -> 2
- net /MODE: track 21.4 -> 31.5 mm, vias 0 -> 2
- net /DN: track 21.7 -> 16.8 mm
- net Net-(R201-Pad1): track 17.0 -> 19.4 mm, vias 3 -> 1
- net GND: track 164.0 -> 163.0 mm
- net /SDA: track 31.6 -> 30.7 mm
- net /SWDCLK: track 96.6 -> 95.7 mm
- net Net-(U202-Pad39): track 0.00 -> 0.80 mm
- net Net-(U202-Pad38): track 0.00 -> 0.80 mm
- net Net-(U202-Pad40): track 0.00 -> 0.73 mm
- net /SCL: track 24.3 -> 23.8 mm
Other:
- board text added: "CLK"
- board text added: "DI-Lambda UNO v1.7"
- board text added: "GND"
- board text added: "IO"
- board text added: "RST"
- board text added: "VCC"
- board text removed: "DI-Lambda UNO v1.6"
