File: DI-Lambda-UNO/DI-Lambda-UNO-top-cover/DI-Lambda-UNO-top-cover.kicad_pcb (KiCad board)
At the start: 2 copper layers, 38.2 x 68.5 mm, 7 parts, among them J12 Conn_01x05, J13 Conn_01x11, J5 Conn_01x11, SW2 SW_BLANK, SW3 SW_SAMPLE, SW4 SW_MODE, U1 LCD_1.44_ST7735

Commit message: Version 1.6
Parts:
- removed J12: Conn_01x05, Connector_PinHeader_2.54mm:PinHeader_1x05_P2.54mm_Vertical_SMD_Pin1Left
- removed J13, J5: Conn_01x11, Connector_PinHeader_2.54mm:PinHeader_1x11_P2.54mm_Vertical_SMD_Pin1Left
- added MK1: Mounting_Hole, MountingHole:MountingHole_3.2mm_M3, F.Cu at (134.6, 44.5)
- added MK2: Mounting_Hole, MountingHole:MountingHole_3.2mm_M3, F.Cu at (166.2, 44.5)
- added MK3: Mounting_Hole, MountingHole:MountingHole_3.2mm_M3, F.Cu at (139.0, 96.1)
- added MK4: Mounting_Hole, MountingHole:MountingHole_3.2mm_M3, F.Cu at (161.8, 96.1)
- added MK5: Mounting_Hole, DI-Lambda-module-tabs:Button_mounts_x3, F.Cu at (150.4, 44.5)
- added TP1: Test_Point, TestPoint:TestPoint_Pad_D1.0mm, B.Cu at (150.4, 43.0)
- SW2, SW3, SW4: footprint MountingHole:MountingHole_4.3mm_M4 -> DI-Lambda-module-tabs:Button-cutout
- moved U1 10.5 mm to (150.4, 64.1)
- moved SW3 3.16 mm to (160.4, 52.0), turned to 0 degrees
- moved SW4 3.16 mm to (140.4, 52.0), turned to 0 degrees
- moved SW2 3.00 mm to (150.4, 52.0), turned to 0 degrees
Routing:
- net GND: track 2.51 -> 0.00 mm
Other:
- board size 38.2 x 68.5 mm -> 38.2 x 58.4 mm
- net class Default: clearance 0.2 -> 0.15; trace_width 0.25 -> 0.15; via_dia 0.8 -> 0.6; via_drill 0.4 -> 0.3
- net class POWER added: clearance 0.2, trace_width 0.3, via_dia 0.6, via_drill 0.3
- rule pad_to_mask_clearance: 0.2 -> 0.07
- rule trace_clearance: 0.2 -> 0.15
- rule trace_min: 0.2 -> 0.15
- board text added: "BLANK"
- board text added: "DI-Lambda UNO v1.6"
- board text added: "MODE"
- board text added: "SAMPLE"
- board text removed: "Blank"
- board text removed: "DI-Lambda UNO v1.5"
- board text removed: "Mode"
- board text removed: "Sample"

Commit message: More missing fotprints
Parts:
- moved TP1 151.6 mm to (3.30, 6.10)
- moved SW2 137.9 mm to (19.1, 9.80)
- moved SW3 137.9 mm to (29.1, 9.80)
- moved MK5 137.8 mm to (19.1, 2.50)
- moved SW4 137.8 mm to (9.10, 10.0)
- moved MK3 137.6 mm to (7.70, 54.9)
- moved MK1 137.6 mm to (3.30, 3.30)
- moved MK2 137.6 mm to (34.9, 3.30)
- moved MK4 137.6 mm to (30.5, 54.9)
- moved U1 137.6 mm to (19.1, 22.9)
Other:
- board text added: "DI-Lambda UNO v1.7"
- board text removed: "DI-Lambda UNO v1.6"
Changed lines of the file:
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@@
-(kicad_pcb (version 20171130) (host pcbnew "(2018-01-22 revision c702646)-master")
+(kicad_pcb (version 20171130) (host pcbnew "(5.0.0-rc2-dev-425-g1663627)")
   (general
     (thickness 1.6)
@@
     (pad_drill 0)
     (pad_to_mask_clearance 0.07)
-    (aux_axis_origin 131.255 41.17)
-    (grid_origin 131.255 41.17)
+    (aux_axis_origin 0 0)
     (visible_elements FFFFFF7F)
     (pcbplotparams
@@
       (drillshape 0)
       (scaleselection 1)
-      (outputdirectory DI-Lambda-UNO-top-cover-v1.6-gerbers-2018-mar-26))
+      (outputdirectory ""))
   )
   (net 0 "")
@@
   )
   (module TestPoint:TestPoint_Pad_D1.0mm (layer B.Cu)
-    (at 150.355 42.97)
+    (at 3.3 6.1)
     (descr "SMD pad as test Point, diameter 1.0mm")
     (tags "test point SMD pad")
@@
   )
   (module MountingHole:MountingHole_3.2mm_M3 (layer F.Cu)
-    (at 161.755 96.07)
+    (at 30.5 54.9)
     (descr "Mounting Hole 3.2mm, no annular, M3")
     (tags "mounting hole 3.2mm no annular m3")
@@
   )
   (module MountingHole:MountingHole_3.2mm_M3 (layer F.Cu)
-    (at 138.955 96.07)
+    (at 7.7 54.9)
     (descr "Mounting Hole 3.2mm, no annular, M3")
     (tags "mounting hole 3.2mm no annular m3")
@@
   )
   (module MountingHole:MountingHole_3.2mm_M3 (layer F.Cu)
-    (at 166.155 44.47)
+    (at 34.9 3.3)
     (descr "Mounting Hole 3.2mm, no annular, M3")
     (tags "mounting hole 3.2mm no annular m3")
@@
   )
   (module MountingHole:MountingHole_3.2mm_M3 (layer F.Cu)
-    (at 134.555 44.47)
+    (at 3.3 3.3)
     (descr "Mounting Hole 3.2mm, no annular, M3")
     (tags "mounting hole 3.2mm no annular m3")
@@
   )
   (module DI-Lambda-module-tabs:Button-cutout (layer B.Cu)
-    (at 140.355 51.97)
+    (at 9.1 10)
     (fp_text reference SW4 (at 0 -0.5) (layer B.SilkS) hide
       (effects (font (size 1 1) (thickness 0.15)) (justify mirror))
@@
   )
   (module DI-Lambda-module-tabs:Button-cutout (layer B.Cu)
-    (at 160.355 51.97)
+    (at 29.1 9.8)
     (fp_text reference SW3 (at 0 -0.5) (layer B.SilkS) hide
       (effects (font (size 1 1) (thickness 0.15)) (justify mirror))
@@
   )
   (module DI-Lambda-module-tabs:Button-cutout (layer B.Cu)
-    (at 150.355 51.97)
+    (at 19.1 9.8)
     (fp_text reference SW2 (at 0 -0.5) (layer B.SilkS) hide
       (effects (font (size 1 1) (thickness 0.15)) (justify mirror))
@@
   )
   (module LCD:LCD_1.44_ST7735-CUTOUT (layer B.Cu)
-    (at 150.405 64.07)
+    (at 19.15 22.9)
     (fp_text reference U1 (at 0 -11.5) (layer B.SilkS) hide
       (effects (font (size 1 1) (thickness 0.15)) (justify mirror))
@@
   )
   (module DI-Lambda-module-tabs:Button_mounts_x3 (layer F.Cu)
-    (at 150.355 44.47)
+    (at 19.1 2.5)
     (fp_text reference MK5 (at 0 6) (layer F.SilkS) hide
       (effects (font (size 1 1) (thickness 0.15)))
@@
       (effects (font (size 1 1) (thickness 0.15)))
     )
-    (pad "" np_thru_hole oval (at 10 0) (size 1.5 1) (drill oval 1.5 1) (layers *.Cu *.Mask))
-    (pad "" np_thru_hole oval (at -10 0) (size 1.5 1) (drill oval 1.5 1) (layers *.Cu *.Mask))
-    (pad "" np_thru_hole oval (at 0 0) (size 1.5 1) (drill oval 1.5 1) (layers *.Cu *.Mask))
+    (pad "" np_thru_hole circle (at 10 0) (size 2.5 2.5) (drill 2.5) (layers *.Cu *.Mask))
+    (pad "" np_thru_hole circle (at -10 0) (size 2.5 2.5) (drill 2.5) (layers *.Cu *.Mask))
+    (pad "" np_thru_hole circle (at 0 0) (size 2.5 2.5) (drill 2.5) (layers *.Cu *.Mask))
   )
   (dimension 10.8 (width 0.3) (layer Eco1.User)
@@
     (arrow2b (pts (xy 174.655 41.17) (xy 175.241421 42.296504)))
   )
-  (gr_line (start 140.355 59.17) (end 140.355 62.17) (layer F.SilkS) (width 0.2))
-  (gr_line (start 150.355 59.17) (end 150.355 62.17) (layer F.SilkS) (width 0.2))
-  (gr_line (start 160.355 59.17) (end 160.355 62.17) (layer F.SilkS) (width 0.2))
-  (gr_text MODE (at 140.355 57.47 180) (layer F.SilkS)
+  (gr_line (start 9.1 18) (end 9.1 21) (layer F.SilkS) (width 0.2))
+  (gr_line (start 19.1 18) (end 19.1 21) (layer F.SilkS) (width 0.2))
+  (gr_line (start 29.1 18) (end 29.1 21) (layer F.SilkS) (width 0.2))
+  (gr_text MODE (at 9.1 16.3 180) (layer F.SilkS)
     (effects (font (size 1.5 1.5) (thickness 0.3)))
   )
-  (gr_text SAMPLE (at 150.255 57.47 180) (layer F.SilkS)
+  (gr_text SAMPLE (at 19 16.3 180) (layer F.SilkS)
     (effects (font (size 1.5 1.5) (thickness 0.3)))
   )
-  (gr_text BLANK (at 160.355 57.47 180) (layer F.SilkS)
+  (gr_text BLANK (at 29.1 16.3 180) (layer F.SilkS)
     (effects (font (size 1.5 1.5) (thickness 0.3)))
   )
-  (gr_line (start 137.355 62.87) (end 137.355 89.97) (layer F.SilkS) (width 0.2))
-  (gr_line (start 163.455 62.87) (end 137.355 62.87) (layer F.SilkS) (width 0.2))
-  (gr_line (start 163.455 89.97) (end 163.455 62.87) (layer F.SilkS) (width 0.2))
-  (gr_line (start 137.355 89.97) (end 163.455 89.97) (layer F.SilkS) (width 0.2))
-  (gr_circle (center 138.955 96.07) (end 141.855 96.07) (layer F.SilkS) (width 0.2))
-  (gr_circle (center 161.755 96.07) (end 164.655 96.07) (layer F.SilkS) (width 0.2))
-  (gr_circle (center 166.155 44.47) (end 169.055 44.47) (layer F.SilkS) (width 0.2))
-  (gr_circle (center 134.555 44.47) (end 137.455 44.47) (layer F.SilkS) (width 0.2))
+  (gr_line (start 6.1 21.7) (end 6.1 48.8) (layer F.SilkS) (width 0.2))
+  (gr_line (start 32.2 21.7) (end 6.1 21.7) (layer F.SilkS) (width 0.2))
+  (gr_line (start 32.2 48.8) (end 32.2 21.7) (layer F.SilkS) (width 0.2))
+  (gr_line (start 6.1 48.8) (end 32.2 48.8) (layer F.SilkS) (width 0.2))
+  (gr_circle (center 7.7 54.9) (end 10.6 54.9) (layer F.SilkS) (width 0.2))
+  (gr_circle (center 30.5 54.9) (end 33.4 54.9) (layer F.SilkS) (width 0.2))
+  (gr_circle (center 34.9 3.3) (end 37.8 3.3) (layer F.SilkS) (width 0.2))
+  (gr_circle (center 3.3 3.3) (end 6.2 3.3) (layer F.SilkS) (width 0.2))
   (dimension 11.8 (width 0.3) (layer Eco1.User)
     (gr_text "11.800 mm" (at 117.805 47.07 90) (layer Eco1.User)
@@
     (arrow2b (pts (xy 119.155 52.97) (xy 118.568579 51.843496)))
   )
-  (gr_arc (start 166.155 96.27) (end 166.155 99.57) (angle -90) (layer Edge.Cuts) (width 0.1))
-  (gr_arc (start 134.555 96.27) (end 131.255 96.27) (angle -90) (layer Edge.Cuts) (width 0.1))
-  (gr_arc (start 166.155 44.47) (end 169.455 44.47) (angle -90) (layer Edge.Cuts) (width 0.1))
+  (gr_arc (start 34.9 55.1) (end 34.9 58.4) (angle -90) (layer Edge.Cuts) (width 0.1))
+  (gr_arc (start 3.3 55.1) (end 0 55.1) (angle -90) (layer Edge.Cuts) (width 0.1))
+  (gr_arc (start 34.9 3.3) (end 38.2 3.3) (angle -90) (layer Edge.Cuts) (width 0.1))
   (dimension 10 (width 0.3) (layer Eco1.User)
     (gr_text "10.000 mm" (at 155.35939 46.674907) (layer Eco1.User)
@@
     (arrow2b (pts (xy 169.455 170.87) (xy 168.328496 171.456421)))
   )
-  (gr_text "DI-Lambda UNO v1.6" (at 133.455 75.57 90) (layer B.Mask)
+  (gr_text "DI-Lambda UNO v1.7" (at 3.2 33.1 90) (layer B.Mask)
     (effects (font (size 1.5 1.5) (thickness 0.3)) (justify mirror))
   )
@@
     (arrow2b (pts (xy 131.255 31.47) (xy 132.381504 30.883579)))
   )
-  (gr_arc (start 134.555 44.47) (end 134.555 41.17) (angle -90) (layer Edge.Cuts) (width 0.1))
-  (gr_line (start 169.455 44.47) (end 169.455 96.27) (layer Edge.Cuts) (width 0.1))
-  (gr_line (start 134.555 41.17) (end 166.155 41.17) (layer Edge.Cuts) (width 0.1))
-  (gr_line (start 131.255 96.27) (end 131.255 44.47) (layer Edge.Cuts) (width 0.1))
-  (gr_line (start 166.155 99.57) (end 134.555 99.57) (layer Edge.Cuts) (width 0.1))
-  (via (at 150.355 42.97) (size 0.6) (drill 0.3) (layers F.Cu B.Cu) (net 1))
+  (gr_arc (start 3.3 3.3) (end 3.3 0) (angle -90) (layer Edge.Cuts) (width 0.1))
+  (gr_line (start 38.2 3.3) (end 38.2 55.1) (layer Edge.Cuts) (width 0.1))
+  (gr_line (start 3.3 0) (end 34.9 0) (layer Edge.Cuts) (width 0.1))
+  (gr_line (start 0 55.1) (end 0 3.3) (layer Edge.Cuts) (width 0.1))
+  (gr_line (start 34.9 58.4) (end 3.3 58.4) (layer Edge.Cuts) (width 0.1))
+  (via (at 5.4 4.3) (size 0.6) (drill 0.3) (layers F.Cu B.Cu) (net 1))
   (zone (net 1) (net_name GND) (layer F.Cu) (hatch edge 0.508)
     (connect_pads (clearance 0.508))
@@
     (polygon
       (pts
-        (xy 131.155 35.97) (xy 169.655 35.97) (xy 169.505 170.57) (xy 130.905 170.77)
+        (xy -0.1 -5.2) (xy 38.4 -5.2) (xy 38.5 59.2) (xy -0.1 59.4)
       )
     )
@@
     (polygon
       (pts
-        (xy 131.155 35.97) (xy 169.655 35.97) (xy 169.505 170.27) (xy 130.905 170.47)
+        (xy -0.1 -5.2) (xy 38.4 -5.2) (xy 38.3 59) (xy -0.3 59.2)
       )
     )
